Commit message: 7

File: src/coppelia_control/urdf/panda.urdf (robot description, URDF)
Before this commit: robot panda, 12 links, 11 joints
Links:
- removed link panda_hand
- removed link panda_leftfinger
- removed link panda_link0
- removed link panda_link1
- removed link panda_link2
- removed link panda_link3
- removed link panda_link4
- removed link panda_link5
- removed link panda_link6
- removed link panda_link7
- removed link panda_link8
- removed link panda_rightfinger
- added link FrankaGripper, mass 0.23000000417233; collision mesh filename=package://coppelia_control/urdf/mesh/panda_FrankaGripper_co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; collision mesh filename=package://coppelia_control/urdf/mesh/panda_FrankaGripper_co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
- added link leftFinger, mass 0.125; collision mesh filename=package://coppelia_control/urdf/mesh/panda_leftFinger_coll_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; collision mesh filename=package://coppelia_control/urdf/mesh/panda_leftFinger_coll_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
- added link leftPad, mass 0.125; collision mesh filename=package://coppelia_control/urdf/mesh/panda_leftPad_coll_1.d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; visual mesh filename=package://coppelia_control/urdf/mesh/panda_leftPad_visible_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
- added link link2_resp, mass 4.9706840515137; collision mesh filename=package://coppelia_control/urdf/mesh/panda_link2_resp_coll_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; collision mesh filename=package://coppelia_control/urdf/mesh/panda_link2_resp_coll_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
- added link link3_resp, mass 0.64692598581314; collision mesh filename=package://coppelia_control/urdf/mesh/panda_link3_resp_coll_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; collision mesh filename=package://coppelia_control/urdf/mesh/panda_link3_resp_coll_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
- added link link4_resp, mass 3.2286040782928; collision mesh filename=package://coppelia_control/urdf/mesh/panda_link4_resp_coll_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; collision mesh filename=package://coppelia_control/urdf/mesh/panda_link4_resp_coll_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
- added link link5_resp, mass 3.5878949165344; collision mesh filename=package://coppelia_control/urdf/mesh/panda_link5_resp_coll_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; collision mesh filename=package://coppelia_control/urdf/mesh/panda_link5_resp_coll_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
- added link link6_resp, mass 1.2259459495544; collision mesh filename=package://coppelia_control/urdf/mesh/panda_link6_resp_coll_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; collision mesh filename=package://coppelia_control/urdf/mesh/panda_link6_resp_coll_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
- added link link7_resp, mass 1.6665550470352; collision mesh filename=package://coppelia_control/urdf/mesh/panda_link7_resp_coll_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; collision mesh filename=package://coppelia_control/urdf/mesh/panda_link7_resp_coll_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
- added link link8_resp, mass 0.73552197217941; collision cylinder length=0.0095007419586182 radius=0.030879393219948; collision cylinder length=0.045800685882568 radius=0.043132938444614
- added link rightFinger, mass 0.125; collision mesh filename=package://coppelia_control/urdf/mesh/panda_rightFinger_coll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; collision mesh filename=package://coppelia_control/urdf/mesh/panda_rightFinger_coll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
- added link rightPad, mass 0.125; collision mesh filename=package://coppelia_control/urdf/mesh/panda_rightPad_coll_1.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; visual mesh filename=package://coppelia_control/urdf/mesh/panda_rightPad_visible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
- added link robot_base; collision mesh filename=package://coppelia_control/urdf/mesh/panda_robot_base_coll_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; visual mesh filename=package://coppelia_control/urdf/mesh/panda_link_vis_1.dae
Joints:
- removed joint panda_finger_joint1
- removed joint panda_finger_joint2
- removed joint panda_hand_joint
- removed joint panda_joint1
- removed joint panda_joint2
- removed joint panda_joint3
- removed joint panda_joint4
- removed joint panda_joint5
- removed joint panda_joint6
- removed joint panda_joint7
- removed joint panda_joint8
- added joint centerJoint: type prismatic, parent FrankaGripper, child leftFinger, origin xyz=0.000168 0.001495 0.074931 rpy=-1.571080 3.141812 3.141556, axis 0 0 1, limit lower=0.0 upper=0.041000001132488 effort=20.0 velocity=0.10000000149012
- added joint connection: type fixed, parent link8_resp, child FrankaGripper, origin xyz=-0.000271 0.000012 0.107001 rpy=3.141593 3.141593 -3.141592, axis 0 0 1
- added joint joint: type revolute, parent robot_base, child link2_resp, origin xyz=-0.349729 -0.074988 0.000000 rpy=-3.141593 3.141593 -3.141593, axis 0 0 1, limit lower=-2.8972465991974 upper=2.8972465991974 effort=87.0 velocity=2.1749997138977
- added joint joint_2: type revolute, parent link2_resp, child link3_resp, origin xyz=-0.000000 -0.000000 0.333000 rpy=1.570796 3.141593 3.141593, axis 0 0 1, limit lower=-1.7627825737 upper=1.7627825737 effort=87.0 velocity=2.1749997138977
- added joint joint_3: type revolute, parent link3_resp, child link4_resp, origin xyz=-0.000000 0.000000 0.000000 rpy=-1.570797 3.141593 -3.141593, axis 0 0 1, limit lower=-2.8972465991974 upper=2.8972465991974 effort=87.0 velocity=2.1749997138977
- added joint joint_4: type revolute, parent link4_resp, child link5_resp, origin xyz=0.082500 -0.000000 0.316000 rpy=-1.570796 3.141593 -3.141592, axis 0 0 1, limit lower=-3.0019662380219 upper=0.0 effort=87.0 velocity=2.1749997138977
- added joint joint_5: type revolute, parent link5_resp, child link6_resp, origin xyz=-0.055513 0.388820 -0.000000 rpy=1.570796 3.141593 3.071779, axis 0 0 1, limit lower=-2.8972465991974 upper=2.8972465991974 effort=12.0 velocity=2.610000371933
- added joint joint_6: type revolute, parent link6_resp, child link7_resp, origin xyz=-0.000000 -0.000000 0.000000 rpy=-1.570796 3.141593 -3.141593, axis 0 0 1, limit lower=-0.017453292384744 upper=3.7524577584118 effort=12.0 velocity=2.610000371933
- added joint joint_7: type revolute, parent link7_resp, child link8_resp, origin xyz=0.088000 0.000000 -0.000000 rpy=-1.570796 3.141592 3.141593, axis 0 0 1, limit lower=-2.8972465991974 upper=2.8972465991974 effort=12.0 velocity=2.610000371933
- added joint leftFingerPad_connection: type fixed, parent leftFinger, child leftPad, origin xyz=0.000028 0.000055 0.006728 rpy=-0.000001 3.141593 -1.570796, axis 0 0 1
- added joint openCloseJoint: type prismatic, parent leftFinger, child rightFinger, origin xyz=-0.000000 -0.000000 -0.000000 rpy=0.000033 3.141592 0.000000, axis 0 0 1, limit lower=0.0 upper=0.082000002264977 effort=20.0 velocity=10.0
- added joint rightFingerPad_connection: type fixed, parent rightFinger, child rightPad, origin xyz=-0.000102 0.000143 0.006578 rpy=0.000034 3.124728 1.574869, axis 0 0 1
